Commit message: send changes to github

File: urdf/jaguar.urdf (robot description, URDF)
Before this commit: robot jaguar_robot, 4 links, 3 joints
Links:
- removed link imu_link
- removed link os_sensor
- removed link zed2_camera_center
- added link gnss
- added link imu
Joints:
- removed joint os_sensor_joint
- removed joint zed2_camera_joint
- added joint gnss: type fixed, parent base_link, child gnss, origin xyz=0.5 0.55 1.9 rpy=0 0 0
- joint imu_joint: child imu_link -> imu; origin xyz=0.14653 0 0.34964 rpy=0 0 0 -> xyz=0.64 -0.15 1.64 rpy=0 0 0
